File: UnitLevelShift.kicad_sch (KiCad schematic)
At the start: 13 parts, among them J1 Conn_01x04_Pin, J2 Conn_01x04_Pin, Q1 2N7002, Q2 2N7002, U1 XC6206PxxxMR

Commit message: Changed LED to optional mounting.
Parts:
- D1: footprint LED_SMD:LED_0603_1608Metric -> LED_THT:LED_D3.0mm; now not fitted
- R5: footprint Resistor_SMD:R_0402_1005Metric -> Resistor_THT:R_Axial_DIN0204_L3.6mm_D1.6mm_P2.54mm_Vertical; now not fitted
